File: hardware/mark-I/telemetry-motherboard/telemetry_mark_I.kicad_pcb (KiCad board)
At the start: 2 copper layers, 112.2 x 142.8 mm, 101 parts, among them J1 Power, J10 5V_BUS, J11 12V_BUS, J12 24V_BUS, J13 Conn_01x02_Socket, J14 Conn_01x02_Socket, J15 Conn_01x02_Socket, J16 Conn_01x02_Socket, J17 BMS_Header, J2 PWM, J3 Analog, J4 PWM, J5 Analog, J6 Communication, J7 Digital, J8 Input_Terminal, J9 Temp_Sensor_Header, U2 ACS712xLCTR-05B, U4 AOZ1284PI, U6 ACS712xLCTR-05B, U7 ACS712xLCTR-05B, U8 ACS712xLCTR-05B

Commit message: Changed routes
Routing:
- net Net-(U4-COMP): track 0.00 -> 102.6 mm, vias 0 -> 1
- net 24V_MEASS: track 0.00 -> 65.1 mm, vias 0 -> 1
Changed lines of the file:
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@@
 		(layer "Edge.Cuts")
+	)
+	(segment
+		(start 100.025 133.525)
+		(end 100 133.5)
+		(width 0.25)
+		(layer "F.Cu")
+		(net "24V_MEASS")
+	)
+	(segment
+		(start 100.025 138.235)
+		(end 100.025 133.525)
+		(width 0.25)
+		(layer "F.Cu")
+		(net "24V_MEASS")
+	)
+	(via
+		(at 100 133.5)
+		(size 0.6)
+		(drill 0.4)
+		(layers "F.Cu" "B.Cu")
+		(net "24V_MEASS")
+	)
+	(segment
+		(start 132.75 133.5)
+		(end 152.25 114)
+		(width 0.25)
+		(layer "B.Cu")
+		(net "24V_MEASS")
+	)
+	(segment
+		(start 100 133.5)
+		(end 132.75 133.5)
+		(width 0.25)
+		(layer "B.Cu")
+		(net "24V_MEASS")
+	)
+	(segment
+		(start 107.75 170.9375)
+		(end 107.75 172.5)
+		(width 0.25)
+		(layer "F.Cu")
+		(net "Net-(U4-COMP)")
+	)
+	(segment
+		(start 106.3175 169.505)
+		(end 107.75 170.9375)
+		(width 0.25)
+		(layer "F.Cu")
+		(net "Net-(U4-COMP)")
+	)
+	(via
+		(at 107.75 172.5)
+		(size 0.6)
+		(drill 0.4)
+		(layers "F.Cu" "B.Cu")
+		(net "Net-(U4-COMP)")
+	)
+	(segment
+		(start 107.75 164.841928)
+		(end 135.85 136.741928)
+		(width 0.25)
+		(layer "B.Cu")
+		(net "Net-(U4-COMP)")
+	)
+	(segment
+		(start 152.7 113.813604)
+		(end 152.436396 113.55)
+		(width 0.25)
+		(layer "B.Cu")
+		(net "Net-(U4-COMP)")
+	)
+	(segment
+		(start 135.85 131.036396)
+		(end 152.7 114.186396)
+		(width 0.25)
+		(layer "B.Cu")
+		(net "Net-(U4-COMP)")
+	)
+	(segment
+		(start 149.45 113.55)
+		(end 136.5 126.5)
+		(width 0.25)
+		(layer "B.Cu")
+		(net "Net-(U4-COMP)")
+	)
+	(segment
+		(start 152.7 114.186396)
+		(end 152.7 113.813604)
+		(width 0.25)
+		(layer "B.Cu")
+		(net "Net-(U4-COMP)")
+	)
+	(segment
+		(start 107.75 172.5)
+		(end 107.75 164.841928)
+		(width 0.25)
+		(layer "B.Cu")
+		(net "Net-(U4-COMP)")
+	)
+	(segment
+		(start 152.436396 113.55)
+		(end 149.45 113.55)
+		(width 0.25)
+		(layer "B.Cu")
+		(net "Net-(U4-COMP)")
+	)
+	(segment
+		(start 135.85 136.741928)
+		(end 135.85 131.036396)
+		(width 0.25)
+		(layer "B.Cu")
+		(net "Net-(U4-COMP)")
 	)
 	(embedded_fonts no)
