File: hardware/bms/bms/bms/bms.kicad_sch (KiCad schematic)
At the start: 24 parts, among them J1 OUTPUT, J2 INPUT_CELL, J3 INPUT_LOGIC, J4 Conn_01x02_Pin, Q1 Q_NPN_BEC

Commit message: New commit
Parts:
- removed J2: INPUT_CELL, Connector_PinHeader_2.54mm:PinHeader_1x05_P2.54mm_Vertical, symbol Connector:Conn_01x05_Pin
- removed J4: Conn_01x02_Pin, TerminalBlock_Phoenix:TerminalBlock_Phoenix_MKDS-1-2-3.81_1x02_P3.81mm_Horizontal, symbol Connector:Conn_01x02_Pin
- added J4: INPUT_CELL1, Connector_PinHeader_2.54mm:PinHeader_1x04_P2.54mm_Vertical, symbol Connector:Conn_01x04_Pin
- added J5: Screw_Terminal_01x02, TerminalBlock_Phoenix:TerminalBlock_Phoenix_MKDS-1,5-2-5.08_1x02_P5.08mm_Horizontal, symbol Connector:Screw_Terminal_01x02
Connections:
- net 5V: now also J5.1 (Pin_1)
- net GND: now also J5.2 (Pin_2)
- net RAW_CELL1: now also J4.1 (Pin_1)
- net RAW_CELL2: now also J4.2 (Pin_2)
- net RAW_CELL3: now also J4.3 (Pin_3)
- net RAW_CELL4: now also J4.4 (Pin_4)

Commit message: PDB Revised
Parts:
- removed J3: INPUT_LOGIC, Connector_PinHeader_2.54mm:PinHeader_1x05_P2.54mm_Vertical, symbol Connector:Conn_01x05_Pin
- removed J4: INPUT_CELL1, Connector_PinHeader_2.54mm:PinHeader_1x04_P2.54mm_Vertical, symbol Connector:Conn_01x04_Pin
- removed J5: Screw_Terminal_01x02, TerminalBlock_Phoenix:TerminalBlock_Phoenix_MKDS-1,5-2-5.08_1x02_P5.08mm_Horizontal, symbol Connector:Screw_Terminal_01x02
- added J2: Conn_01x05_Pin, Connector_JST:JST_EH_B5B-EH-A_1x05_P2.50mm_Vertical, symbol Connector:Conn_01x05_Pin
- added J3: Conn_01x06_Pin, Connector_JST:JST_EH_B6B-EH-A_1x06_P2.50mm_Vertical, symbol Connector:Conn_01x06_Pin
- J1: footprint Connector_PinHeader_2.54mm:PinHeader_1x04_P2.54mm_Vertical -> Connector_JST:JST_EH_B4B-EH-A_1x04_P2.50mm_Vertical
- RTOP12, RTOP13, RTOP14, RTOP9: value 330 -> 680
Connections:
- net 5V: now also J3.6 (Pin_6)
- net BUZZER_GATE: now also J3.5 (Pin_5)
- net GND: now also J2.5 (Pin_5)
- net LED1: now also J3.1 (Pin_1)
- net LED2: now also J3.2 (Pin_2)
- net LED3: now also J3.3 (Pin_3)
- net LED4: now also J3.4 (Pin_4)
- net RAW_CELL1: now also J2.1 (Pin_1)
- net RAW_CELL2: now also J2.2 (Pin_2)
- net RAW_CELL3: now also J2.3 (Pin_3)
- net RAW_CELL4: now also J2.4 (Pin_4)
Other:
- moved on the sheet: BZ1, D1, D2, D3, D4, J1, Q1, RBOTT5, RBOTT6, RBOTT7, RBOTT8, RTOP10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

Commit message: Added Sensors & LCD
Parts:
- D1, D2, D3, D4: footprint LED_SMD:LED_1206_3216Metric -> LED_SMD:LED_0805_2012Metric
- RTOP1: renamed from RTOP5; value 47K -> 27K
- RTOP2: renamed from RTOP7; value 47K -> 27K
- RTOP3: renamed from RTOP6; value 47K -> 27K
- RTOP4: renamed from RTOP8; value 47K -> 27K
- renumbered RBOTT5 to RBOT1, RBOTT7 to RBOT2, RBOTT6 to RBOT3, RBOTT8 to RBOT4, RTOP10 to RBZR1, RTOP11 to RBZRPULL1, RTOP9 to RLED1, RTOP13 to RLED2, RTOP14 to RLED3, RTOP12 to RLED4
Connections:
- net LED1: no longer RLED1.1
- net LED2: no longer RLED2.1
- net LED3: no longer RLED3.1
- net LED4: no longer RLED4.1
- new net RLED1: RLED1.1
- new net RLED2: RLED2.1
- new net RLED3: RLED3.1
- new net RLED4: RLED4.1
Changed lines of the file:
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@@
 		)
 	)
-	(label "LED4"
+	(label "RLED4"
 		(at 166.37 123.19 0)
 		(effects
@@
 		)
 	)
-	(label "LED2"
+	(label "RLED2"
 		(at 132.08 135.89 0)
 		(effects
@@
 		)
 	)
-	(label "LED1"
+	(label "RLED1"
 		(at 132.08 123.19 0)
 		(effects
@@
 		)
 	)
-	(label "LED3"
+	(label "RLED3"
 		(at 166.37 135.89 0)
 		(effects
@@
 		(dnp no)
 		(fields_autoplaced yes)
-		(property "Reference" "RBOTT6"
+		(property "Reference" "RBOT3"
 			(at 69.85 124.4599 0)
 			(show_name no)
@@
 			(project "bms"
 				(path "/cb811605-a31a-48ea-ac3c-b6e14ef2e5ea"
-					(reference "RBOTT6")
+					(reference "RBOT3")
 					(unit 1)
 				)
@@
 			)
 		)
-		(property "Footprint" "LED_SMD:LED_1206_3216Metric"
+		(property "Footprint" "LED_SMD:LED_0805_2012Metric"
 			(at 147.32 123.19 0)
 			(hide yes)
@@
 		(dnp no)
 		(fields_autoplaced yes)
-		(property "Reference" "RTOP14"
+		(property "Reference" "RLED3"
 			(at 172.72 129.54 90)
 			(show_name no)
@@
 			(project "bms"
 				(path "/cb811605-a31a-48ea-ac3c-b6e14ef2e5ea"
-					(reference "RTOP14")
+					(reference "RLED3")
 					(unit 1)
 				)
@@
 		(dnp no)
 		(fields_autoplaced yes)
-		(property "Reference" "RTOP6"
+		(property "Reference" "RTOP3"
 			(at 69.85 114.2999 0)
 			(show_name no)
@@
 			)
 		)
-		(property "Value" "47K"
+		(property "Value" "27K"
 			(at 69.85 116.8399 0)
 			(show_name no)
@@
 			(project "bms"
 				(path "/cb811605-a31a-48ea-ac3c-b6e14ef2e5ea"
-					(reference "RTOP6")
+					(reference "RTOP3")
 					(unit 1)
 				)
@@
 		(dnp no)
 		(fields_autoplaced yes)
-		(property "Reference" "RTOP13"
+		(property "Reference" "RLED2"
 			(at 138.43 129.54 90)
 			(show_name no)
@@
 			(project "bms"
 				(path "/cb811605-a31a-48ea-ac3c-b6e14ef2e5ea"
-					(reference "RTOP13")
+					(reference "RLED2")
 					(unit 1)
 				)
@@
 			)
 		)
-		(property "Footprint" "LED_SMD:LED_1206_3216Metric"
+		(property "Footprint" "LED_SMD:LED_0805_2012Metric"
 			(at 181.61 123.19 0)
 			(hide yes)
@@
 		(dnp no)
 		(fields_autoplaced yes)
-		(property "Reference" "RBOTT8"
+		(property "Reference" "RBOT4"
 			(at 96.52 124.4599 0)
 			(show_name no)
@@
 			(project "bms"
 				(path "/cb811605-a31a-48ea-ac3c-b6e14ef2e5ea"
-					(reference "RBOTT8")
+					(reference "RBOT4")
 					(unit 1)
 				)
@@
 			)
 		)
-		(property "Footprint" "LED_SMD:LED_1206_3216Metric"
+		(property "Footprint" "LED_SMD:LED_0805_2012Metric"
 			(at 181.61 135.89 0)
 			(hide yes)
@@
 		(dnp no)
 		(fields_autoplaced yes)
-		(property "Reference" "RBOTT7"
+		(property "Reference" "RBOT2"
 			(at 96.52 87.6299 0)
 			(show_name no)
@@
 			(project "bms"
 				(path "/cb811605-a31a-48ea-ac3c-b6e14ef2e5ea"
-					(reference "RBOTT7")
+					(reference "RBOT2")
 					(unit 1)
 				)
@@
 		(in_pos_files yes)
 		(dnp no)
-		(property "Reference" "RTOP11"
+		(property "Reference" "RBZRPULL1"
 			(at 149.86 96.5201 0)
 			(show_name no)
@@
 			(project "bms"
 				(path "/cb811605-a31a-48ea-ac3c-b6e14ef2e5ea"
-					(reference "RTOP11")
+					(reference "RBZRPULL1")
 					(unit 1)
 				)
@@
 		(dnp no)
 		(fields_autoplaced yes)
-		(property "Reference" "RTOP9"
+		(property "Reference" "RLED1"
 			(at 138.43 116.84 90)
 			(show_name no)
@@
 			(project "bms"
 				(path "/cb811605-a31a-48ea-ac3c-b6e14ef2e5ea"
-					(reference "RTOP9")
+					(reference "RLED1")
 					(unit 1)
 				)
@@
 		(dnp no)
 		(fields_autoplaced yes)
-		(property "Reference" "RTOP8"
+		(property "Reference" "RTOP4"
 			(at 96.52 114.2999 0)
 			(show_name no)
@@
 			)
 		)
-		(property "Value" "47K"
+		(property "Value" "27K"
 			(at 96.52 116.8399 0)
 			(show_name no)
@@
 			(project "bms"
 				(path "/cb811605-a31a-48ea-ac3c-b6e14ef2e5ea"
-					(reference "RTOP8")
+					(reference "RTOP4")
 					(unit 1)
 				)
@@
 		(dnp no)
 		(fields_autoplaced yes)
-		(property "Reference" "RTOP5"
+		(property "Reference" "RTOP1"
 			(at 69.85 77.4699 0)
 			(show_name no)
@@
 			)
 		)
-		(property "Value" "47K"
+		(property "Value" "27K"
 			(at 69.85 80.0099 0)
 			(show_name no)
@@
 			(project "bms"
 				(path "/cb811605-a31a-48ea-ac3c-b6e14ef2e5ea"
-					(reference "RTOP5")
+					(reference "RTOP1")
 					(unit 1)
 				)
@@
 		(dnp no)
 		(fields_autoplaced yes)
-		(property "Reference" "RTOP7"
+		(property "Reference" "RTOP2"
 			(at 96.52 77.4699 0)
 			(show_name no)
@@
 			)
 		)
-		(property "Value" "47K"
+		(property "Value" "27K"
 			(at 96.52 80.0099 0)
 			(show_name no)
@@
 			(project "bms"
 				(path "/cb811605-a31a-48ea-ac3c-b6e14ef2e5ea"
-					(reference "RTOP7")
+					(reference "RTOP2")
 					(unit 1)
 				)
@@
 		(dnp no)
 		(fields_autoplaced yes)
-		(property "Reference" "RBOTT5"
+		(property "Reference" "RBOT1"
 			(at 69.85 87.6299 0)
 			(show_name no)
@@
 			(project "bms"
 				(path "/cb811605-a31a-48ea-ac3c-b6e14ef2e5ea"
-					(reference "RBOTT5")
+					(reference "RBOT1")
 					(unit 1)
 				)
@@
 		(in_pos_files yes)
 		(dnp no)
-		(property "Reference" "RTOP10"
+		(property "Reference" "RBZR1"
 			(at 143.5099 85.09 0)
 			(show_name no)
@@
 			(project "bms"
 				(path "/cb811605-a31a-48ea-ac3c-b6e14ef2e5ea"
-					(reference "RTOP10")
+					(reference "RBZR1")
 					(unit 1)
 				)
@@
 		(dnp no)
 		(fields_autoplaced yes)
-		(property "Reference" "RTOP12"
+		(property "Reference" "RLED4"
 			(at 172.72 116.84 90)
 			(show_name no)
@@
 			(project "bms"
 				(path "/cb811605-a31a-48ea-ac3c-b6e14ef2e5ea"
-					(reference "RTOP12")
+					(reference "RLED4")
 					(unit 1)
 				)
@@
 			)
 		)
-		(property "Footprint" "LED_SMD:LED_1206_3216Metric"
+		(property "Footprint" "LED_SMD:LED_0805_2012Metric"
 			(at 147.32 135.89 0)
 			(hide yes)
