File: hardware/mark-II/telemetry-motherboard/telemetry_mark_I.kicad_pcb (KiCad board)
At the start: 2 copper layers, 112.2 x 142.8 mm, 101 parts, among them J1 Power, J10 5V_BUS, J11 12V_BUS, J12 24V_BUS, J13 Conn_01x02_Socket, J14 Conn_01x02_Socket, J15 Conn_01x02_Socket, J16 Conn_01x02_Socket, J17 BMS_Header, J2 PWM, J3 Analog, J4 PWM, J5 Analog, J6 Communication, J7 Digital, J8 Input_Terminal, J9 Temp_Sensor_Header, U2 ACS712xLCTR-05B, U4 AOZ1284PI, U6 ACS712xLCTR-05B, U7 ACS712xLCTR-05B, U8 ACS712xLCTR-05B

Commit message: New commit
Parts:
- removed C11: 30u, Capacitor_THT:CP_Radial_D5.0mm_P2.00mm
- removed C12, C17, C19, C27, C28: 10u, Capacitor_SMD:C_0603_1608Metric_Pad1.08x0.95mm_HandSolder
- removed C14: 4.7n, Capacitor_SMD:C_0603_1608Metric_Pad1.08x0.95mm_HandSolder
- removed C18, C20: 0.3n, Capacitor_SMD:C_0603_1608Metric_Pad1.08x0.95mm_HandSolder
- removed C22, C23: 1n, Capacitor_SMD:C_0603_1608Metric_Pad1.08x0.95mm_HandSolder
- removed C24, C25: 100n, Capacitor_SMD:C_0603_1608Metric_Pad1.08x0.95mm_HandSolder
- removed C5, C6: 68n, Capacitor_SMD:C_0603_1608Metric_Pad1.08x0.95mm_HandSolder
- removed C7: 33n, Capacitor_SMD:C_0603_1608Metric_Pad1.08x0.95mm_HandSolder
- removed C9: 4.7u, Capacitor_SMD:C_0603_1608Metric_Pad1.08x0.95mm_HandSolder
- removed D6, D7: SS54, Diode_SMD:D_SMA
- removed L1: 6.8u, Inductor_SMD:L_0603_1608Metric_Pad1.05x0.95mm_HandSolder
- removed L2, L3: 22u, Inductor_SMD:L_12x12mm_H8mm
- removed MH3: MountingHole_3.2mm, Arduino_MountingHole:MountingHole_3.2mm
- removed R13: 27.4k, Resistor_SMD:R_0603_1608Metric_Pad0.98x0.95mm_HandSolder
- removed R15: 43.2k, Resistor_SMD:R_0603_1608Metric_Pad0.98x0.95mm_HandSolder
- removed R16, R26: 105k, Resistor_SMD:R_0603_1608Metric_Pad0.98x0.95mm_HandSolder
- removed R17, R18: 47k, Resistor_SMD:R_0603_1608Metric_Pad0.98x0.95mm_HandSolder
- removed R19, R21: 680k, Resistor_SMD:R_0603_1608Metric_Pad0.98x0.95mm_HandSolder
- removed R2: 20k, Resistor_SMD:R_0603_1608Metric_Pad0.98x0.95mm_HandSolder
- removed R20, R22: 100k, Resistor_SMD:R_0603_1608Metric_Pad0.98x0.95mm_HandSolder
- removed R23: 52.3k, Resistor_SMD:R_0603_1608Metric_Pad0.98x0.95mm_HandSolder
- removed R24: 10k, Resistor_SMD:R_0603_1608Metric_Pad0.98x0.95mm_HandSolder
- removed R27: 7.5k, Resistor_SMD:R_0603_1608Metric_Pad0.98x0.95mm_HandSolder
- removed R3: 120k, Resistor_SMD:R_0603_1608Metric_Pad0.98x0.95mm_HandSolder
- removed R8: 2.8M, Resistor_SMD:R_0603_1608Metric_Pad0.98x0.95mm_HandSolder
- removed U4: AOZ1284PI, Package_SO:SOIC-8-1EP_3.9x4.9mm_P1.27mm_EP2.71x3.7mm
- added C16: 100nF, Capacitor_SMD:C_0805_2012Metric, F.Cu at (289.2, 165.8)
- added C21: 1nF, Capacitor_SMD:C_0805_2012Metric, F.Cu at (289.2, 168.8)
- added C26: 100nF, Capacitor_SMD:C_0805_2012Metric, F.Cu at (289.2, 136.6)
- added C29: 1nF, Capacitor_SMD:C_0805_2012Metric, F.Cu at (289.2, 139.6)
- added C30: 100nF, Capacitor_SMD:C_0805_2012Metric, F.Cu at (289.2, 151.2)
- added C31: 1nF, Capacitor_SMD:C_0805_2012Metric, F.Cu at (289.2, 154.2)
- added C32: 100nF, Capacitor_SMD:C_0805_2012Metric, F.Cu at (300.1, 180.4)
- added C33: 1nF, Capacitor_SMD:C_0805_2012Metric, F.Cu at (300.1, 183.4)
- added D10: LED, LED_SMD:LED_0805_2012Metric, F.Cu at (304.5, 180.4)
- added D5: LED, LED_SMD:LED_0805_2012Metric, F.Cu at (293.6, 165.8)
- added D8: LED, LED_SMD:LED_0805_2012Metric, F.Cu at (293.6, 136.6)
- added D9: LED, LED_SMD:LED_0805_2012Metric, F.Cu at (293.6, 151.2)
- added R10: 1k, Resistor_SMD:R_0805_2012Metric, F.Cu at (293.6, 154.2)
- added R11: 1k, Resistor_SMD:R_0805_2012Metric, F.Cu at (304.5, 183.4)
- added R7: 1k, Resistor_SMD:R_0805_2012Metric, F.Cu at (293.6, 168.8)
- added R9: 1k, Resistor_SMD:R_0805_2012Metric, F.Cu at (293.6, 139.6)
- added U10: ACS712xLCTR-05B, Package_SO:SOIC-8_3.9x4.9mm_P1.27mm, F.Cu at (291.2, 131.9)
- added U11: ACS712xLCTR-05B, Package_SO:SOIC-8_3.9x4.9mm_P1.27mm, F.Cu at (291.2, 146.5)
- added U12: ACS712xLCTR-05B, Package_SO:SOIC-8_3.9x4.9mm_P1.27mm, F.Cu at (302.1, 175.7)
- added U9: ACS712xLCTR-05B, Package_SO:SOIC-8_3.9x4.9mm_P1.27mm, F.Cu at (291.2, 161.1)
- J10: footprint TerminalBlock_Phoenix:TerminalBlock_Phoenix_MKDS-1,5-8_1x08_P5.00mm_Horizontal -> TerminalBlock_Phoenix:TerminalBlock_Phoenix_MKDS-1,5-8-5.08_1x08_P5.08mm_Horizontal
- J13, J14, J15, J16: footprint Connector_AMASS:AMASS_XT60-F_1x02_P7.20mm_Vertical -> Connector_AMASS:AMASS_XT60PW-F_1x02_P7.20mm_Horizontal
- J8: footprint TerminalBlock_Ningbo-Kagnex:TerminalBlock_Ningbo-Kagnex_HB9500_1x05_P9.5mm -> TerminalBlock_Ningbo-Kagnex:TerminalBlock_Ningbo-Kagnex_HB9500_1x08_P9.5mm
- moved J7 236.2 mm to (322.5, 119.6), turned to 180 degrees
- moved MH6 227.1 mm to (322.6, 71.3), turned to 0 degrees
- moved MH5 224.3 mm to (316.2, 119.6), turned to 0 degrees
- moved H4 214.1 mm to (350.0, 70.0), turned to 180 degrees
- moved J15 212.4 mm to (350.0, 105.0), turned to -90 degrees
- moved J16 202.3 mm to (350.0, 175.0), turned to -90 degrees
- moved H2 192.2 mm to (350.0, 210.0), turned to 180 degrees
- moved J8 186.7 mm to (275.0, 210.0)
- moved J6 183.8 mm to (294.6, 119.6), turned to 90 degrees
- moved J5 181.8 mm to (299.7, 71.3), turned to 90 degrees
- moved J9 172.8 mm to (274.5, 167.2)
- moved J10 152.2 mm to (245.8, 134.7)
- moved J12 152.2 mm to (245.8, 159.0)
- moved J4 142.6 mm to (271.8, 119.6), turned to 90 degrees
- moved J3 136.7 mm to (276.9, 71.3), turned to 90 degrees
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Connections:
- net +12V renamed /+12V
- net +24V renamed /+24V
- J13 pad 1: BATT_MEASS -> /W1_MEASS
- J14 pad 1: BATT_MEASS -> /W2_MEASS
- J15 pad 1: BATT_MEASS -> /W3_MEASS
- J16 pad 1: BATT_MEASS -> /W4_MEASS
Other:
- board size 112.2 x 142.8 mm -> 300 x 160 mm
- copper layers 2 -> 4

Commit message: PDB Revised
Parts:
- removed J10: 5V_BUS, TerminalBlock_Phoenix:TerminalBlock_Phoenix_MKDS-1,5-8-5.08_1x08_P5.08mm_Horizontal
- removed J11: 12V_BUS, TerminalBlock_Phoenix:TerminalBlock_Phoenix_MKDS-1,5-8_1x08_P5.00mm_Horizontal
- removed J12: 24V_BUS, TerminalBlock_Phoenix:TerminalBlock_Phoenix_MKDS-1,5-8_1x08_P5.00mm_Horizontal
- added BZ1: Buzzer, Buzzer_Beeper:Buzzer_12x9.5RM7.6, F.Cu at (433.4, 120.9)
- added C5: C_Polarized, Capacitor_SMD:CP_Elec_8x10.5, F.Cu at (421.0, 267.2)
- added C6: C_Polarized, Capacitor_SMD:CP_Elec_8x10.5, F.Cu at (421.0, 197.0)
- added C7: C_Polarized, Capacitor_SMD:CP_Elec_8x10.5, F.Cu at (173.5, 267.3)
- added C9: C_Polarized, Capacitor_SMD:CP_Elec_8x10.5, F.Cu at (174.0, 197.2)
- added D11: LED, LED_SMD:LED_1206_3216Metric, F.Cu at (427.6, 122.6)
- added D12: LED, LED_SMD:LED_1206_3216Metric, F.Cu at (427.6, 126.0)
- added D6: LED, LED_SMD:LED_1206_3216Metric, F.Cu at (427.6, 115.8)
- added D7: LED, LED_SMD:LED_1206_3216Metric, F.Cu at (427.6, 119.2)
- added J18: Screw_Terminal_01x08, TerminalBlock_Ningbo-Kagnex:TerminalBlock_Ningbo-Kagnex_HB9500_1x08_P9.5mm, F.Cu at (332.2, 291.0)
- added J19: Conn_01x06_Pin, Connector_PinSocket_2.54mm:PinSocket_1x06_P2.54mm_Horizontal, F.Cu at (388.7, 154.5)
- added J20: Screw_Terminal_01x02, TerminalBlock_Phoenix:TerminalBlock_Phoenix_MKDS-1,5-2-5.08_1x02_P5.08mm_Horizontal, F.Cu at (300.6, 191.2)
- added J20: Screw_Terminal_01x02, TerminalBlock_Phoenix:TerminalBlock_Phoenix_MKDS-1,5-2-5.08_1x02_P5.08mm_Horizontal, F.Cu at (302.0, 232.2)
- added J20: Screw_Terminal_01x02, TerminalBlock_Phoenix:TerminalBlock_Phoenix_MKDS-1,5-2-5.08_1x02_P5.08mm_Horizontal, F.Cu at (202.0, 237.2)
- added J20: Screw_Terminal_01x02, TerminalBlock_Phoenix:TerminalBlock_Phoenix_MKDS-1,5-2-5.08_1x02_P5.08mm_Horizontal, F.Cu at (202.9, 196.0)
- added J21: Screw_Terminal_01x04, Connector_Phoenix_MC:PhoenixContact_MCV_1,5_4-GF-3.81_1x04_P3.81mm_Vertical_ThreadedFlange_MountHole, F.Cu at (348.8, 171.8)
- added Q1: Q_NPN_BEC, Package_TO_SOT_SMD:SOT-23, F.Cu at (437.4, 129.9)
- added RTOP10: 1k, Resistor_SMD:R_0805_2012Metric, F.Cu at (422.5, 118.6)
- added RTOP11: 10k, Resistor_SMD:R_0805_2012Metric, F.Cu at (422.5, 121.5)
- added RTOP12: 680, Resistor_SMD:R_0805_2012Metric, F.Cu at (422.5, 124.5)
- added RTOP13: 680, Resistor_SMD:R_0805_2012Metric, F.Cu at (422.5, 127.4)
- added RTOP14: 680, Resistor_SMD:R_0805_2012Metric, F.Cu at (422.5, 130.4)
- added RTOP9: 680, Resistor_SMD:R_0805_2012Metric, F.Cu at (422.5, 115.6)
- added U1: ~, PDB:ArduinoMega, F.Cu at (203.2, 117.5)
- added U13: ~, PDB:Untitled_3, F.Cu at (422.0, 147.3)
- added U3: ~, PDB:Untitled, F.Cu at (251.2, 186.5)
- added U4: ~, PDB:Untitled_1, F.Cu at (354.8, 225.0)
- added U5: ~, PDB:24Converter, F.Cu at (252.0, 237.2)
- J8: value Input_Terminal -> INPUT_CELL1; footprint TerminalBlock_Ningbo-Kagnex:TerminalBlock_Ningbo-Kagnex_HB9500_1x08_P9.5mm -> Connector_PinHeader_2.54mm:PinHeader_1x04_P2.54mm_Vertical
- RBOTT5, RBOTT6, RBOTT7, RBOTT8, RTOP5, RTOP6, RTOP7, RTOP8: footprint Resistor_SMD:R_0603_1608Metric_Pad0.98x0.95mm_HandSolder -> Resistor_SMD:R_0805_2012Metric
- moved D8 184.3 mm to (185.1, 285.6), turned to -90 degrees
- moved R9 183.7 mm to (182.1, 285.5), turned to -90 degrees
- moved U10 179.0 mm to (183.6, 275.0), turned to -90 degrees
- moved C26 178.1 mm to (185.1, 281.1), turned to -90 degrees
- moved C29 177.5 mm to (182.1, 281.1), turned to -90 degrees
- moved RBOTT1 160.8 mm to (414.6, 117.4), turned to -90 degrees
- moved RBOTT2 159.2 mm to (412.1, 117.4), turned to -90 degrees
- moved RBOTT3 157.7 mm to (409.6, 117.4), turned to -90 degrees
- moved RBOTT4 156.2 mm to (407.1, 117.4), turned to -90 degrees
- moved RBOTT7 155.4 mm to (414.6, 121.8), turned to -90 degrees
- moved RBOTT5 154.8 mm to (404.6, 117.4), turned to -90 degrees
- moved RBOTT8 153.7 mm to (412.1, 121.8), turned to -90 degrees
- moved RBOTT6 153.5 mm to (402.1, 117.4), turned to -90 degrees
- moved RTOP1 152.1 mm to (409.6, 121.8), turned to -90 degrees
- moved RTOP2 150.6 mm to (407.1, 121.8), turned to -90 degrees
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Connections:
- J13 pad 1: /W1_MEASS -> GND
- J13 pad 2: GND -> /W1_MEASS
- J14 pad 1: /W2_MEASS -> GND
- J14 pad 2: GND -> /W2_MEASS
- J15 pad 1: /W3_MEASS -> GND
- J15 pad 2: GND -> /W3_MEASS
- J16 pad 1: /W4_MEASS -> GND
- J16 pad 2: GND -> /W4_MEASS
- J17 pad 1: RAW_CELL1 -> /RAW_CELL1
- J17 pad 2: RAW_CELL2 -> /RAW_CELL2
- J17 pad 3: RAW_CELL3 -> /RAW_CELL3
- J17 pad 4: RAW_CELL4 -> /RAW_CELL4
- J8 pad 1: /RAW_BATT(15-5) -> RAW_CELL1
- J8 pad 2: /RAW_BATT(15-12) -> RAW_CELL2
- J8 pad 3: /RAW_BATT(15-24) -> RAW_CELL3
- J8 pad 4: /RAW_BATT(15-ESCs) -> RAW_CELL4
- RBOTT5 pad 1: /MEASS_CELL1 -> /BMS/MEASS_CELL1
- RBOTT6 pad 1: /MEASS_CELL3 -> /BMS/MEASS_CELL3
- RBOTT7 pad 1: /MEASS_CELL2 -> /BMS/MEASS_CELL2
- RBOTT8 pad 1: /MEASS_CELL4 -> /BMS/MEASS_CELL4
- RTOP5 pad 2: /MEASS_CELL1 -> /BMS/MEASS_CELL1
- RTOP6 pad 2: /MEASS_CELL3 -> /BMS/MEASS_CELL3
- RTOP7 pad 2: /MEASS_CELL2 -> /BMS/MEASS_CELL2
- RTOP8 pad 2: /MEASS_CELL4 -> /BMS/MEASS_CELL4
Routing:
- net GND: track 0.00 -> 12.9 mm, vias 0 -> 26
- net +5V: track 0.00 -> 8.15 mm
- net Net-(D9-A): track 0.00 -> 3.02 mm
- net Net-(D10-A): track 0.00 -> 3.02 mm
- net Net-(U11-FILTER): track 0.00 -> 2.93 mm
- net Net-(U12-FILTER): track 0.00 -> 2.79 mm
- added copper zone on F.Cu, net /RAW_BATT(15-W1)
- added copper zone on F.Cu, net /RAW_BATT(15-W2)
- added copper zone on F.Cu, net /RAW_BATT(15-W3)
- added copper zone on F.Cu, net /RAW_BATT(15-W4)
- added copper zone on F.Cu, net /W1_MEASS
- added copper zone on F.Cu, net /W2_MEASS
- added copper zone on F.Cu, net /W3_MEASS
- added copper zone on F.Cu, net /W4_MEASS
- added copper zone on F.Cu, net GND
- added copper zone on In1.Cu, net GND
Other:
- board size 300 x 160 mm -> 300 x 240 mm
- board text added: "GND"

Commit message: Added 3D Models
Parts:
- added J18: Screw_Terminal_01x08, TerminalBlock_Ningbo-Kagnex:TerminalBlock_Ningbo-Kagnex_HB9500_1x08_P9.5mm, F.Cu at (344.8, 96.4)
Routing:
- net unconnected-(J20-Pin_2-Pad2): track 0.00 -> 112.3 mm
- added copper zone on F.Cu, net +5V

Commit message: Added Sensors & LCD
Parts:
- removed the J18 at (344.8, 96.4)
- removed J8: INPUT_CELL1, Connector_PinHeader_2.54mm:PinHeader_1x04_P2.54mm_Vertical
- added J13: Conn_01x02_Socket, Connector_AMASS:AMASS_XT60PW-F_1x02_P7.20mm_Horizontal, F.Cu at (358.8, 80.3)
- added J13: Conn_01x02_Socket, Connector_AMASS:AMASS_XT60PW-F_1x02_P7.20mm_Horizontal, F.Cu at (304.1, 80.8)
- added J13: Conn_01x02_Socket, Connector_AMASS:AMASS_XT60PW-F_1x02_P7.20mm_Horizontal, F.Cu at (407.6, 79.0)
- J9: footprint Connector_PinHeader_2.54mm:PinHeader_1x03_P2.54mm_Vertical -> Connector_JST:JST_EH_B3B-EH-A_1x03_P2.50mm_Vertical
- moved U13 248.6 mm to (174.2, 167.0), turned to 180 degrees
- moved J19 181.3 mm to (207.5, 159.8), turned to 0 degrees
- moved J9 30.1 mm to (403.0, 158.8)
Routing:
- net unconnected-(J20-Pin_2-Pad2): track 112.3 -> 0.00 mm
- removed copper zone on F.Cu, net +5V
